File: componentes1.sch (EAGLE design)
At the start: 14 parts, among them IC1 LD117AS33TR, K1 CQ1-12V, T1 BC337, U1 DS1307Z, X1 32.768KHZ

Commit message: se agrega board
Parts:
- added C4, C5, C6, C7: (no value), rcl:C-EU050-025X075
- added H1, H2, H3, H4: MOUNT-HOLE3.2, holes:MOUNT-HOLE3.2
- added Q1: (no value), crystal:CRYSTALHC49S
- added R3, R6: (no value), rcl:R-EU_0204/7
- added S2: (no value), switch-omron:40-XX
- added U2: ATMEGA32U4-AU, ATMEGA32U4-AU:ATMEGA32U4-AU
- added U3: RFM95W-868S2, RFM95W-868S2:RFM95W-868S2
- added X2: MINI-USB-32005-201, con-cypressindustries:MINI-USB-32005-201
- added X3: BU-SMA-V, con-coax:BU-SMA-V
Connections:
- new net ANT: U3.ANT, X3.1
- new net ID: X2.4
- new net N$10: U2.AREF
- new net N$11: U2.XTAL1
- new net N$12: U2.PB0
- new net N$13: U2.PB1
- new net N$14: U2.PB2
- new net N$15: U2.PB3
- new net N$16: U2.PB4
- new net N$17: U2.PB5
- new net N$18: U2.PB6
- new net N$19: U2.PB7
- new net N$20: U2.PD0
- new net N$21: U2.PD1
- new net N$22: U2.PD2
- new net N$23: U2.PD3
- new net N$24: U2.PD4
- new net N$25: U2.PD5
- new net N$26: U2.PD6
- new net N$27: U2.PD7
- new net N$28: U2.UCAP
- new net N$29: R3.1, U2.D-
- new net N$30: U2.PF7
- new net N$31: U2.PF6
- new net N$32: U2.PF5
- new net N$33: U2.PF4
- new net N$34: U2.PF1
- new net N$35: U2.PF0
- new net N$36: U2.PE6
- new net N$37: U2.PC7
- new net N$38: U2.PC6
- new net N$39: U2.XTAL2
- new net N$40: R3.2, X2.2
- new net N$41: U3.RESET
- new net N$42: R6.2, X2.3
- new net N$43: R6.1, U2.D+
- new net N$44: U2.PE2
- new net N$45: U3.MISO
- new net N$46: U3.SCK
- new net N$47: U3.NSS
- new net N$49: U3.DIO5
- new net N$50: U3.DIO3
- new net N$51: U3.DIO4
- new net N$52: U3.DIO0
- new net N$53: U3.DIO1
- new net N$54: U3.DIO2
- new net N$58: U3.MOSI
- new net N$8: U2.VBUS
- new net RESET: S2.P, S2.P1, U2.!RESET
- new net XTAL1: C6.2, Q1.1
- new net XTAL2: C7.2, Q1.2
- net 3.3V: now also C4.1, C5.1, U2.AVCC, U2.UVCC, U2.VCC, U3.3_3V
- net GND: now also C4.2, C5.2, C6.1, C7.1, S2.S, S2.S1, U2.GND, U2.UGND, U3.GND, U3.GND@1, U3.GND@2, X2.5, X3.2
- net VCC: now also X2.1

Commit message: sos
Changed lines of the file:
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@@
 <part name="C3" library="rcl" library_urn="urn:adsk.eagle:library:334" deviceset="C-EU" device="050-025X075" package3d_urn="urn:adsk.eagle:package:23637/1"/>
 <part name="FRAME2" library="frames" library_urn="urn:adsk.eagle:library:229" deviceset="A4L-LOC" device=""/>
-<part name="FRAME3" library="frames" library_urn="urn:adsk.eagle:library:229" deviceset="A4L-LOC" device=""/>
 <part name="U2" library="ATMEGA32U4-AU" deviceset="ATMEGA32U4-AU" device=""/>
 <part name="U3" library="RFM95W-868S2" deviceset="RFM95W-868S2" device=""/>
@@
 </nets>
 </sheet>
-<sheet>
-<plain>
-</plain>
-<instances>
-<instance part="FRAME3" gate="G$1" x="-10.16" y="-22.86" smashed="yes">
-<attribute name="DRAWING_NAME" x="207.01" y="-7.62" size="2.54" layer="94"/>
-<attribute name="LAST_DATE_TIME" x="207.01" y="-12.7" size="2.286" layer="94"/>
-<attribute name="SHEET" x="220.345" y="-17.78" size="2.54" layer="94"/>
-</instance>
-</instances>
-<busses>
-</busses>
-<nets>
-</nets>
-</sheet>
