File: iot_pcb.brd (EAGLE design)
At the start: 80 x 80 mm, 16 parts, among them U1 RFM95W-868S2, U2 ATMEGA32U4-AU, X1 MINI-USB-32005-201, X2 BU-SMA-V

Commit message: xfabo no c muera
Parts:
- removed C2: (no value), rcl:C050-025X075
- added BAT1: BATTERY_1236_C, Itead_BP_110825.lbr:BATTERY_1236_C
- added C10, C11, C6, C7, C8, C9: (no value), rcl:C050-025X075
- added C5: 100nF, rcl:C0603
- added D1: 1N4446, diode:DO35-10
- added IC1: LD117AS33TR, v-reg:SOT223
- added K1: CQ1-12V, relay:CQ1
- added LED1: PC56H19_V0, led:PC56H19_V0
- added R1, R4, R5, R6: (no value), rcl:0207/10
- added R7, R8: (no value), rcl:0204/7
- added T1: BC337, transistor:TO92
- added U3: DS1307Z, SparkFun-Clocks:SO08-0.15
- added X3: 32.768KHZ, adafruit:XTAL3215
- moved Q1 53.2 mm to (25.5, 68.0)
- moved C3 52.5 mm to (25.5, 74.0)
- moved C4 52.0 mm to (25.5, 61.5)
- moved C1 30.3 mm to (68.0, 61.0)
- moved U2 18.6 mm to (44.5, 71.0)
- moved X2 18.1 mm to (75.0, 27.0)
- moved S2 12.0 mm to (28.5, 50.0)
- moved X1 10.7 mm to (8.00, 58.5)
- moved R2 9.43 mm to (17.5, 69.5)
- moved R3 9.43 mm to (14.0, 69.5)
- moved U1 8.32 mm to (64.0, 42.0)
Connections:
- removed net 3.3V: C1.1, C2.1, U1.13, U2.14, U2.2, U2.24, U2.34, U2.44
- removed net N$36: U2.16
- removed net N$4 (its old number): U2.17
- new net 12V: C6.1, IC1.3
- new net 5V: C8.2, R7.1, R8.2
- new net AVCC: C11.1, U2.24, U2.44
- new net N$2: BAT1.+, U3.3
- new net N$3: U3.1, X3.P$2
- new net N$37: U3.2, X3.P$1
- new net N$38: D1.A, K1.2, T1.3
- new net N$39: D1.C, K1.1
- new net N$40: R1.2, R4.2, T1.2
- new net N$41: LED1.2, LED1.4, R8.1
- new net SCL: R5.1, U3.6
- new net SDA: R6.2, U3.5
- new net SQW: U3.7
- new net TIER: C6.2, C7.2, IC1.1
- new net TIERR: R4.1
- new net UVCC: C10.2, U2.2
- new net VIN: R1.1
- net GND: now also BAT1.-, C10.1, C11.2, C5.1, C8.1, C9.1, LED1.1, LED1.3, T1.1, U3.4; no longer C2.2
- net N$7: now also K1.NO
- net N$9: now also K1.C
- net RESET: now also R7.2
- net VCC: now also C1.1, C5.2, C7.1, C9.2, IC1.4, R5.2, R6.1, U1.13, U2.14, U2.34, U3.8
- net XTAL1: now also U2.17
- net XTAL2: now also U2.16

Commit message: sos
Parts:
- added C12, C2: (no value), rcl:C050-025X075
- added R9: (no value), rcl:0204/7
Connections:
- removed net 5V: C8.2, R7.1, R8.2
- removed net N$25: R2.1, U2.3
- removed net N$42: R3.2, X1.3
- removed net N$43: R3.1, U2.4
- removed net UVCC: C10.2, U2.2
- new net D+: R2.1, U2.4
- new net D-: R3.1, U2.3
- new net VBUS: C12.2, U2.7, X1.1
- net AVCC: now also C10.2, C8.2, C9.2, R7.1, R8.2, U2.14, U2.2, U2.34
- net GND: now also C12.1, C2.2, R9.1
- net N$1: now also C2.1, U2.6; no longer U2.7
- net N$23: now also R3.2, X1.2; no longer U2.6
- net N$24: now also X1.3; no longer X1.2
- net N$33: now also R9.2
- net VCC: no longer C9.2, U2.14, U2.34, X1.1
Changed lines of the file:
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@@
 <attribute name="VALUE" x="0.75" y="-35.5" size="1.27" layer="27" ratio="6"/>
+</element>
+<element name="C2" library="rcl" library_urn="urn:adsk.eagle:library:334" package="C050-025X075" package3d_urn="urn:adsk.eagle:package:23637/1" value="" x="4" y="-39.5" smashed="yes">
+<attribute name="NAME" x="0.571" y="-37.849" size="1.27" layer="25" ratio="10"/>
+<attribute name="POPULARITY" value="29" x="4" y="-39.5" size="1.778" layer="27" display="off"/>
+<attribute name="SPICEPREFIX" value="C" x="4" y="-39.5" size="1.778" layer="27" display="off"/>
+<attribute name="VALUE" x="0.571" y="-42.294" size="1.27" layer="27" ratio="10"/>
+</element>
+<element name="C12" library="rcl" library_urn="urn:adsk.eagle:library:334" package="C050-025X075" package3d_urn="urn:adsk.eagle:package:23637/1" value="" x="4" y="-44.5" smashed="yes">
+<attribute name="NAME" x="0.571" y="-42.849" size="1.27" layer="25" ratio="10"/>
+<attribute name="POPULARITY" value="29" x="4" y="-44.5" size="1.778" layer="27" display="off"/>
+<attribute name="SPICEPREFIX" value="C" x="4" y="-44.5" size="1.778" layer="27" display="off"/>
+<attribute name="VALUE" x="0.571" y="-47.294" size="1.27" layer="27" ratio="10"/>
+</element>
+<element name="R9" library="rcl" library_urn="urn:adsk.eagle:library:334" package="0204/7" package3d_urn="urn:adsk.eagle:package:23498/2" value="" x="4.5" y="-49" smashed="yes">
+<attribute name="NAME" x="1.96" y="-47.7046" size="0.9906" layer="25" ratio="10"/>
+<attribute name="POPULARITY" value="79" x="4.5" y="-49" size="1.778" layer="27" display="off"/>
+<attribute name="SPICEPREFIX" value="R" x="4.5" y="-49" size="1.778" layer="27" display="off"/>
+<attribute name="VALUE" x="2.8744" y="-49.4826" size="0.9906" layer="27" ratio="10"/>
 </element>
 </elements>
 <signals>
-<signal name="N$1">
-<contactref element="U2" pad="7"/>
-</signal>
 <signal name="N$5">
 <contactref element="U2" pad="8"/>
@@
 <contactref element="U2" pad="27"/>
 </signal>
-<signal name="N$23">
-<contactref element="U2" pad="6"/>
-</signal>
-<signal name="N$25">
-<contactref element="U2" pad="3"/>
-<contactref element="R2" pad="1"/>
-<wire x1="17.5" y1="73.31" x2="38.6" y2="73.4" width="0" layer="19" extent="1-1"/>
-</signal>
 <signal name="N$26">
 <contactref element="U2" pad="36"/>
@@
 <contactref element="U2" pad="31"/>
 </signal>
-<signal name="N$42">
-<contactref element="X1" pad="3"/>
-<contactref element="R3" pad="2"/>
-<wire x1="11" y1="58.5" x2="14" y2="73.31" width="0" layer="19" extent="1-1"/>
-</signal>
 <signal name="N$45">
 <contactref element="U1" pad="2"/>
@@
 <signal name="N$58">
 <contactref element="U1" pad="3"/>
-</signal>
-<signal name="N$24">
-<contactref element="X1" pad="2"/>
-<contactref element="R2" pad="2"/>
-<wire x1="11" y1="59.3" x2="17.5" y2="65.69" width="0" layer="19" extent="1-1"/>
-</signal>
-<signal name="N$43">
-<contactref element="U2" pad="4"/>
-<contactref element="R3" pad="1"/>
-<wire x1="14" y1="65.69" x2="38.6" y2="72.6" width="0" layer="19" extent="1-1"/>
 </signal>
 <signal name="N$21">
@@
 <vertex x="80" y="80"/>
 </polygon>
-<contactref element="X1" pad="5"/>
 <contactref element="S2" pad="1"/>
 <contactref element="S2" pad="2"/>
@@
 <contactref element="LED1" pad="3"/>
 <contactref element="LED1" pad="1"/>
+<contactref element="X1" pad="5"/>
+<contactref element="C12" pad="1"/>
+<contactref element="C2" pad="2"/>
+<contactref element="R9" pad="1"/>
 <wire x1="56.6" y1="49" x2="68" y2="58.46" width="0" layer="19" extent="1-1"/>
 <wire x1="56.6" y1="35" x2="56.6" y2="49" width="0" layer="19" extent="1-1"/>
@@
 <wire x1="1.49" y1="-31.85" x2="6.54" y2="-19" width="0" layer="19" extent="1-1"/>
 <wire x1="1.49" y1="-33.145" x2="1.49" y2="-31.85" width="0" layer="19" extent="1-1"/>
+<wire x1="6.54" y1="-39.5" x2="1.49" y2="-33.145" width="0" layer="19" extent="1-1"/>
+<wire x1="1.46" y1="-44.5" x2="6.54" y2="-39.5" width="0" layer="19" extent="1-1"/>
+<wire x1="0.69" y1="-49" x2="1.46" y2="-44.5" width="0" layer="19" extent="1-1"/>
 </signal>
 <signal name="ANT">
@@
 <signal name="N$33">
 <contactref element="U2" pad="33"/>
-</signal>
-<signal name="ID">
-<contactref element="X1" pad="4"/>
+<contactref element="R9" pad="2"/>
+<wire x1="8.31" y1="-49" x2="50.4" y2="75" width="0" layer="19" extent="1-1"/>
 </signal>
 <signal name="VCC">
-<contactref element="X1" pad="1"/>
 <contactref element="U3" pad="8"/>
 <contactref element="C5" pad="2"/>
@@
 <contactref element="IC1" pad="4"/>
 <contactref element="C7" pad="1"/>
-<contactref element="C9" pad="2"/>
-<contactref element="U2" pad="34"/>
-<contactref element="U2" pad="14"/>
 <wire x1="63.93" y1="67.1" x2="68" y2="63.54" width="0" layer="19" extent="1-1"/>
 <wire x1="60.93" y1="63.63" x2="63.93" y2="67.1" width="0" layer="19" extent="1-1"/>
-<wire x1="48.5" y1="76.9" x2="60.93" y2="63.63" width="0" layer="19" extent="1-1"/>
-<wire x1="42.1" y1="65.1" x2="48.5" y2="76.9" width="0" layer="19" extent="1-1"/>
 <wire x1="71.4" y1="43" x2="68" y2="63.54" width="0" layer="19" extent="1-1"/>
-<wire x1="11" y1="60.1" x2="42.1" y2="65.1" width="0" layer="19" extent="1-1"/>
-<wire x1="3.45" y1="46.32" x2="11" y2="60.1" width="0" layer="19" extent="1-1"/>
-<wire x1="7.125" y1="42.5" x2="3.45" y2="46.32" width="0" layer="19" extent="1-1"/>
+<wire x1="15.38" y1="39.82" x2="60.93" y2="63.63" width="0" layer="19" extent="1-1"/>
+<wire x1="7.125" y1="42.5" x2="15.38" y2="39.82" width="0" layer="19" extent="1-1"/>
+<wire x1="3.45" y1="46.32" x2="7.125" y2="42.5" width="0" layer="19" extent="1-1"/>
 <wire x1="3.87" y1="38.05" x2="7.125" y2="42.5" width="0" layer="19" extent="1-1"/>
-<wire x1="15.38" y1="39.82" x2="7.125" y2="42.5" width="0" layer="19" extent="1-1"/>
-<wire x1="6.54" y1="-9" x2="3.87" y2="38.05" width="0" layer="19" extent="1-1"/>
 </signal>
 <signal name="N$22">
@@
 </signal>
 <signal name="AVCC">
-<contactref element="C11" pad="1"/>
-<contactref element="U2" pad="24"/>
-<contactref element="U2" pad="44"/>
-<wire x1="40.5" y1="76.9" x2="50.4" y2="67.8" width="0" layer="19" extent="1-1"/>
-<wire x1="1.46" y1="-19" x2="50.4" y2="67.8" width="0" layer="19" extent="1-1"/>
-</signal>
-<signal name="UVCC">
-<contactref element="C10" pad="2"/>
-<contactref element="U2" pad="2"/>
-<wire x1="6.54" y1="-14" x2="38.6" y2="74.2" width="0" layer="19" extent="1-1"/>
-</signal>
-<signal name="5V">
 <contactref element="R7" pad="1"/>
 <contactref element="C8" pad="2"/>
 <contactref element="R8" pad="2"/>
+<contactref element="C9" pad="2"/>
+<contactref element="C10" pad="2"/>
+<contactref element="C11" pad="1"/>
+<contactref element="U2" pad="34"/>
+<contactref element="U2" pad="14"/>
+<contactref element="U2" pad="2"/>
+<contactref element="U2" pad="24"/>
+<contactref element="U2" pad="44"/>
+<wire x1="40.5" y1="76.9" x2="48.5" y2="76.9" width="0" layer="19" extent="1-1"/>
+<wire x1="38.6" y1="74.2" x2="40.5" y2="76.9" width="0" layer="19" extent="1-1"/>
+<wire x1="50.4" y1="67.8" x2="48.5" y2="76.9" width="0" layer="19" extent="1-1"/>
+<wire x1="42.1" y1="65.1" x2="50.4" y2="67.8" width="0" layer="19" extent="1-1"/>
+<wire x1="6.54" y1="-4" x2="42.1" y2="65.1" width="0" layer="19" extent="1-1"/>
+<wire x1="6.54" y1="-9" x2="6.54" y2="-4" width="0" layer="19" extent="1-1"/>
+<wire x1="6.54" y1="-14" x2="6.54" y2="-9" width="0" layer="19" extent="1-1"/>
+<wire x1="1.46" y1="-19" x2="6.54" y2="-14" width="0" layer="19" extent="1-1"/>
+<wire x1="0.69" y1="-23.5" x2="1.46" y2="-19" width="0" layer="19" extent="1-1"/>
 <wire x1="8.31" y1="-27.5" x2="0.69" y2="-23.5" width="0" layer="19" extent="1-1"/>
-<wire x1="6.54" y1="-4" x2="0.69" y2="-23.5" width="0" layer="19" extent="1-1"/>
 </signal>
 <signal name="N$41">
@@
 <wire x1="0.69" y1="-27.5" x2="5.695" y2="-31.85" width="0" layer="19" extent="1-1"/>
 </signal>
+<signal name="VBUS">
+<contactref element="U2" pad="7"/>
+<contactref element="X1" pad="1"/>
+<contactref element="C12" pad="2"/>
+<wire x1="11" y1="60.1" x2="38.6" y2="70.2" width="0" layer="19" extent="1-1"/>
+<wire x1="6.54" y1="-44.5" x2="11" y2="60.1" width="0" layer="19" extent="1-1"/>
+</signal>
+<signal name="D+">
+<contactref element="U2" pad="4"/>
+<contactref element="R2" pad="1"/>
+<wire x1="17.5" y1="73.31" x2="38.6" y2="72.6" width="0" layer="19" extent="1-1"/>
+</signal>
+<signal name="D-">
+<contactref element="U2" pad="3"/>
+<contactref element="R3" pad="1"/>
+<wire x1="14" y1="65.69" x2="38.6" y2="73.4" width="0" layer="19" extent="1-1"/>
+</signal>
+<signal name="N$24">
+<contactref element="X1" pad="3"/>
+<contactref element="R2" pad="2"/>
+<wire x1="11" y1="58.5" x2="17.5" y2="65.69" width="0" layer="19" extent="1-1"/>
+</signal>
+<signal name="ID">
+<contactref element="X1" pad="4"/>
+</signal>
+<signal name="N$23">
+<contactref element="X1" pad="2"/>
+<contactref element="R3" pad="2"/>
+<wire x1="11" y1="59.3" x2="14" y2="73.31" width="0" layer="19" extent="1-1"/>
+</signal>
+<signal name="N$1">
+<contactref element="U2" pad="6"/>
+<contactref element="C2" pad="1"/>
+<wire x1="1.46" y1="-39.5" x2="38.6" y2="71" width="0" layer="19" extent="1-1"/>
+</signal>
 </signals>
