File: iot_pcb.sch (EAGLE design)
At the start: 16 parts, among them U1 RFM95W-868S2, U2 ATMEGA32U4-AU, X1 MINI-USB-32005-201, X2 BU-SMA-V

Commit message: xfabo no c muera
Parts:
- removed C2: (no value), rcl:C-EU050-025X075
- added BAT1: BATTERY_1236_C, Itead_BP_110825.lbr:BATTERY_1236_C
- added C10, C11, C6, C7, C8, C9: (no value), rcl:C-EU050-025X075
- added C5: 100nF, rcl:C-EUC0603
- added D1: 1N4446, diode:1N4446
- added IC1: LD117AS33TR, v-reg:LD117AS33TR
- added K1: CQ1-12V, relay:CQ1-12V
- added LED1: PC56H19_V0, led:PC56H19_V0
- added R1, R4, R5, R6: (no value), rcl:R-EU_0207/10
- added R7, R8: (no value), rcl:R-EU_0204/7
- added T1: BC337, transistor:BC337
- added U3: DS1307Z, SparkFun-Clocks:DS1307Z
- added X3: 32.768KHZ, adafruit:XTAL-3.2X1.5
Connections:
- removed net 3.3V: C1.1, C2.1, U1.3_3V, U2.AVCC, U2.UVCC, U2.VCC
- removed net N$36: U2.XTAL2
- removed net N$4 (its old number): U2.XTAL1
- new net 12V: C6.1, IC1.IN
- new net 5V: C8.2, R7.1, R8.2
- new net AVCC: C11.1, U2.AVCC
- new net N$2: BAT1.+, U3.VBATT
- new net N$3: U3.X1, X3.P$2
- new net N$37: U3.X2, X3.P$1
- new net N$38: D1.A, K11.2, T1.C
- new net N$39: D1.C, K11.1
- new net N$40: R1.2, R4.2, T1.B
- new net N$41: LED1.A, R8.1
- new net SCL: R5.1, U3.SCL
- new net SDA: R6.2, U3.SDA
- new net SQW: U3.SQW
- new net TIER: C6.2, C7.2, IC1.ADJ
- new net TIERR: R4.1
- new net UVCC: C10.2, U2.UVCC
- new net VIN: R1.1
- net GND: now also BAT1.-, C10.1, C11.2, C5.1, C8.1, C9.1, LED1.C, T1.E, U3.GND; no longer C2.2
- net N$7: now also K12.S
- net N$9: now also K12.P
- net RESET: now also R7.2
- net VCC: now also C1.1, C5.2, C7.1, C9.2, IC1.OUT, R5.2, R6.1, U1.3_3V, U2.VCC, U3.VCC
- net XTAL1: now also U2.XTAL1
- net XTAL2: now also U2.XTAL2

Commit message: sos
Parts:
- added C12, C2: (no value), rcl:C-EU050-025X075
- added R9: (no value), rcl:R-EU_0204/7
Connections:
- removed net 5V: C8.2, R7.1, R8.2
- removed net N$25: R2.1, U2.D-
- removed net N$42: R3.2, X1.3
- removed net N$43: R3.1, U2.D+
- removed net UVCC: C10.2, U2.UVCC
- new net D+: R2.1, U2.D+
- new net D-: R3.1, U2.D-
- new net VBUS: C12.2, U2.VBUS, X1.1
- net AVCC: now also C10.2, C8.2, C9.2, R7.1, R8.2, U2.UVCC, U2.VCC
- net GND: now also C12.1, C2.2, R9.1
- net N$1: now also C2.1, U2.UCAP; no longer U2.VBUS
- net N$23: now also R3.2, X1.2; no longer U2.UCAP
- net N$24: now also X1.3; no longer X1.2
- net N$33: now also R9.2
- net VCC: no longer C9.2, U2.VCC, X1.1
Other:
- moved on the sheet: C3, C4, C9, Q1, R2, R3, U2, X1
